Commit message: cell: launch + urdf + scripts

File: cooperative_transport_cell/urdf/fake_base.macro.xacro (robot description, xacro)
@@ -4,8 +4,15 @@
                                             world_frame
                                             create_world:=false
-                                            use_ros2_control:=true">
+                                            use_ros2_control:=true
+                                            *origin">
   <xacro:if value="${create_world}">
     <link name="${world_frame}"/>
   </xacro:if>
+  <link name="${prefix}move_starting_frame"/>
+  <joint name="${prefix}fixed_offset" type="fixed">
+    <xacro:insert_block name="origin"/>
+    <parent link="${world_frame}"/>
+    <child link="${prefix}move_starting_frame"/>
+  </joint>
   <link name="${prefix}linear_x"/>
   <link name="${prefix}linear_y"/>
@@ -13,5 +20,5 @@
   <link name="${prefix}mount_frame"/>
   <joint name="${prefix}joint_x" type="prismatic">
-    <parent link="${world_frame}"/>
+    <parent link="${prefix}move_starting_frame"/>
     <child  link="${prefix}linear_x"/>
     <axis xyz="1 0 0"/>

File: cooperative_transport_cell/urdf/imm.xacro (robot description, xacro)
@@ -8,5 +8,7 @@
   <xacro:arg name="create_world_frame" default="true"/>
   <xacro:arg name="use_PPR"            default="true"/>
-  <!-- <xacro:arg name=""> -->
+  <xacro:arg name="color_base"         default="1.0 0.0 0.0 1.0"/>
+  <xacro:arg name="xyz"                default="0.0 0.0 0.0"/>
+  <xacro:arg name="rpy"                default="0.0 0.0 0.0"/>
 <!--
     ##############
@@ -91,4 +93,7 @@
         <box size="1.0 0.5 0.4" rpy="0 0 0"/>
       </geometry>
+      <material name="colored">
+        <color rgba="$(arg color_base)"/>
+      </material>
     </visual>
   </link>
@@ -103,5 +108,7 @@
                            world_frame="$(arg world_frame)"
                            create_world="$(arg create_world_frame)"
-                           use_ros2_control="true"/>
+                           use_ros2_control="true">
+      <origin xyz="$(arg xyz)" rpy="$(arg rpy)"/>
+    </xacro:fake_base_macro>
     <joint name="$(arg prefix)" type="fixed">
       <parent link="$(arg prefix)mount_frame"/>
